File: PCBA/HumanoidArduino.brd (EAGLE design)
At the start: 105.4 x 75.2 mm, 23 parts, among them IC1 7805TV, J2 22-27-2041-04

Commit message: Continued work on PCBA
Parts:
- added JP10, JP11, JP12, JP13, JP14, JP15, JP16, JP17, JP18, JP19, JP20, JP21, JP22, JP23, JP24, JP25: (no value), jumper:JP2
- added JP9: (no value), jumper:JP1
- added R7: 670R, SparkFun-Passives:0805
- added R8: 330R, SparkFun-Passives:0805
- added S1: (no value), SparkFun-Electromechanical:SWITCH-SPDT_LOCK.007S
- added U$1: P-CHANNEL-MOSFET, GeekAmmo:SOT23-3
- added U$2, U$4: HSMC-C265, SparkFun-Retired:HSMC-C265
- JP1, JP2, JP3, JP4, JP5, JP6, JP7, JP8: device jumper:JP2W -> jumper:JP2
- moved JP8 250.2 mm to (6.35, 31.8), turned to 180 degrees
- moved JP7 236.2 mm to (6.35, 35.6), turned to 180 degrees
- moved JP2 222.2 mm to (6.35, 57.1), turned to 180 degrees
- moved JP6 222.2 mm to (6.35, 39.4), turned to 180 degrees
- moved JP5 190.5 mm to (6.35, 43.2), turned to 180 degrees
- moved JP4 179.1 mm to (6.35, 49.5), turned to 180 degrees
- moved JP3 165.1 mm to (6.35, 53.3), turned to 180 degrees
- moved JP1 137.2 mm to (6.35, 61.0), turned to 180 degrees
- moved R6 129.5 mm to (45.7, 57.1), turned to 270 degrees
- moved R3 128.1 mm to (80.0, 54.6), turned to 90 degrees
- moved R2 126.2 mm to (80.0, 58.4), turned to 90 degrees
- moved R1 124.3 mm to (80.0, 62.2), turned to 90 degrees
- moved R5 120.1 mm to (45.7, 53.3), turned to 270 degrees
- moved R4 110.8 mm to (48.3, 48.3), turned to 270 degrees
- moved U2 96.2 mm to (66.0, 55.9), turned to 90 degrees
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Connections:
- net 12.6V renamed 12.6V_CHG
- net 4.2V renamed 4.2V_CHG
- new net +5V1: JP10.2, JP11.2, JP12.2, JP13.2, JP14.2, JP15.2, JP16.2, JP17.2, JP18.2, JP19.2, JP20.2, JP21.2, JP22.2, JP23.2, JP24.2, JP25.2
- new net 8.4V_CHG: J2.3
- new net 8.4V_IN: JP9.2, S1.2
- new net N$10: JP10.1, R4.4
- new net N$11: JP11.1, R4.3
- new net N$12: JP12.1, R4.2
- new net N$13: JP13.1, R4.1
- new net N$14: JP14.1, R3.4
- new net N$15: JP15.1, R3.3
- new net N$16: JP16.1, R3.2
- new net N$17: JP17.1, R3.1
- new net N$18: JP18.1, R2.4
- new net N$19: JP19.1, R2.3
- new net N$20: JP20.1, R2.2
- new net N$21: JP21.1, R2.1
- new net N$22: JP22.1, R1.4
- new net N$23: JP23.1, R1.3
- new net N$24: JP24.1, R1.2
- new net N$25: JP25.1, R1.1
- new net N$26: S1.3, U$1.2
- new net N$28: R7.1, U$4.A
- new net N$29: R8.1, U$2.A
- new net N$6: JP5.1, R5.4
- new net N$7: JP6.1, R5.3
- new net N$8: JP7.1, R5.2
- new net N$9: JP8.1, R5.1
- net +5V: now also R8.2
- net 8.4V: now also R7.2, U$1.3; no longer J2.3
- net GND: now also JP10.3, JP11.3, JP12.3, JP13.3, JP14.3, JP15.3, JP16.3, JP17.3, JP18.3, JP19.3, JP20.3, JP21.3, JP22.3, JP23.3, JP24.3, JP25.3, JP9.1, U$1.1, U$2.C, U$4.C
- net N$3: now also JP2.1; no longer JP3.1
- net N$4: now also JP3.1; no longer JP4.1
- net N$5: now also JP4.1; no longer JP5.1
Routing:
- net 8.4V: track 66.7 -> 0.00 mm
- net +5V: track 58.0 -> 0.00 mm
- net SCL: track 48.4 -> 0.00 mm
- net SDA: track 48.4 -> 0.00 mm
- net \O\E: track 12.5 -> 0.00 mm

Commit message: more PCBA work
Parts:
- added F1, F10, F11, F12, F13, F14, F15, F16, F17, F18, F19, F2, F20, F21, F22, F23, F24, F25, F26, F3, F4, F5, F6, F7, F8, F9: POLYSWITCH, HumanoidLbr:1206
- added JP26, JP27: JUMPER_3X1_0.1, HumanoidLbr:CONN_3X1_0.1"
- added R10, R9: (no value), SparkFun-Resistors:0603-ARV
- JP1, JP10, JP11, JP12, JP13, JP14, JP15, JP16, JP17, JP18, JP19, JP2, JP20, JP21, JP22, JP23, JP24, JP25, JP3, JP4, JP5, JP6, JP7, JP8: value (none) -> JUMPER_3X1_0.1; device jumper:JP2 -> HumanoidLbr:CONN_3X1_0.1"
- moved JP17 84.2 mm to (14.0, 22.9), turned to 180 degrees
- moved JP16 84.1 mm to (14.0, 25.4), turned to 180 degrees
- moved JP15 84.0 mm to (14.0, 27.9), turned to 180 degrees
- moved JP14 83.9 mm to (14.0, 30.5), turned to 180 degrees
- moved R3 35.4 mm to (45.7, 45.7), turned to 270 degrees
- moved JP13 19.3 mm to (14.0, 33.0)
- moved JP21 19.3 mm to (90.2, 50.8)
- moved JP20 18.2 mm to (90.2, 53.3)
- moved JP12 18.2 mm to (14.0, 35.6)
- moved JP11 17.0 mm to (14.0, 38.1)
- moved JP19 17.0 mm to (90.2, 55.9)
- moved JP22 17.0 mm to (90.2, 48.3)
- moved JP18 15.9 mm to (90.2, 58.4)
- moved JP23 15.9 mm to (90.2, 45.7)
- moved JP10 15.9 mm to (14.0, 40.6)
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Connections:
- removed net +5V1: JP10.2, JP11.2, JP12.2, JP13.2, JP14.2, JP15.2, JP16.2, JP17.2, JP18.2, JP19.2, JP20.2, JP21.2, JP22.2, JP23.2, JP24.2, JP25.2
- new net N$27: F1.P$1, JP1.P$2
- new net N$30: F2.P$1, JP2.P$2
- new net N$31: JP12.P$1, R4.3
- new net N$32: JP13.P$1, R4.4
- new net N$33: JP14.P$1, R3.1
- new net N$34: JP15.P$1, R3.2
- new net N$35: JP16.P$1, R3.3
- new net N$36: JP17.P$1, R3.4
- new net N$38: F21.P$1, JP22.P$2
- new net N$39: F20.P$1, JP21.P$2
- new net N$40: F19.P$1, JP20.P$2
- new net N$41: F18.P$1, JP19.P$2
- new net N$42: F17.P$1, JP18.P$2
- new net N$43: JP18.P$1, R9.8
- new net N$44: JP19.P$1, R9.7
- new net N$45: JP20.P$1, R9.6
- new net N$46: JP21.P$1, R9.5
- new net N$47: JP22.P$1, R10.8
- new net N$48: F22.P$1, JP23.P$2
- new net N$49: F23.P$1, JP24.P$2
- new net N$50: F24.P$1, JP25.P$2
- new net N$51: F25.P$1, JP26.P$2
- new net N$52: F26.P$1, JP27.P$2
- new net N$53: JP23.P$1, R10.7
- new net N$54: JP24.P$1, R10.6
- new net N$55: JP25.P$1, R10.5
- net +5V: now also F1.P$2, F10.P$2, F11.P$2, F12.P$2, F13.P$2, F14.P$2, F15.P$2, F16.P$2, F17.P$2, F18.P$2, F19.P$2, F2.P$2, F20.P$2, F21.P$2, F22.P$2, F23.P$2, F24.P$2, F25.P$2, F26.P$2, F3.P$2, F4.P$2, F5.P$2, F6.P$2, F7.P$2, F8.P$2, F9.P$2; no longer JP1.2, JP2.2, JP3.2, JP4.2, JP5.2, JP6.2, JP7.2, JP8.2
- net GND: now also JP1.P$3, JP18.P$3, JP19.P$3, JP2.P$3, JP20.P$3, JP21.P$3, JP22.P$3, JP23.P$3, JP24.P$3, JP25.P$3, JP26.P$3, JP27.P$3, JP3.P$3, JP4.P$3; no longer JP1.3, JP10.3, JP11.3, JP12.3, JP13.3, JP14.3, JP15.3, JP16.3, JP17.3, JP18.3, JP19.3, JP2.3, JP20.3, JP21.3, JP22.3, JP23.3, JP24.3, JP25.3, JP3.3, JP4.3, JP5.3, JP6.3, JP7.3, JP8.3
- net N$10: now also F14.P$1, JP15.P$2; no longer JP10.1, R4.4
- net N$11: now also F13.P$1, JP14.P$2; no longer JP11.1, R4.3
- net N$12: now also F12.P$1, JP13.P$2; no longer JP12.1, R4.2
- net N$13: now also F11.P$1, JP12.P$2; no longer JP13.1, R4.1
- net N$14: now also F10.P$1, JP11.P$2; no longer JP14.1, R3.4
- net N$15: now also F9.P$1, JP10.P$2; no longer JP15.1, R3.3
- net N$16: now also F8.P$1, JP8.P$2; no longer JP16.1, R3.2
- net N$17: now also F7.P$1, JP7.P$2; no longer JP17.1, R3.1
- net N$18: now also F6.P$1, JP6.P$2; no longer JP18.1, R2.4
- net N$19: now also F5.P$1, JP5.P$2; no longer JP19.1, R2.3
- net N$2: now also JP1.P$1, R6.1; no longer JP1.1, R6.4
- net N$20: now also JP5.P$1, R5.1; no longer JP20.1, R2.2
- net N$21: now also JP6.P$1, R5.2; no longer JP21.1, R2.1
- net N$22: now also JP7.P$1, R5.3; no longer JP22.1, R1.4
- net N$23: now also JP8.P$1, R5.4; no longer JP23.1, R1.3
- net N$24: now also JP10.P$1, R4.1; no longer JP24.1, R1.2
- net N$25: now also JP11.P$1, R4.2; no longer JP25.1, R1.1
- net N$3: now also JP2.P$1, R6.2; no longer JP2.1, R6.3
- net N$4: now also JP3.P$1, R6.3; no longer JP3.1, R6.2
- net N$5: now also JP4.P$1, R6.4; no longer JP4.1, R6.1
- net N$6: now also F3.P$1, JP3.P$2; no longer JP5.1, R5.4
- net N$7: now also F4.P$1, JP4.P$2; no longer JP6.1, R5.3
- net N$8: now also F16.P$1, JP17.P$2; no longer JP7.1, R5.2
- net N$9: now also F15.P$1, JP16.P$2; no longer JP8.1, R5.1
- net PWM0: now also R6.8; no longer R6.5
- net PWM1: now also R6.7; no longer R6.6
- net PWM10: now also R4.6; no longer R4.7
- net PWM11: now also R4.5; no longer R4.8
- net PWM12: now also R3.8
- net PWM13: now also R3.7
- net PWM14: now also R3.6
- net PWM15: now also R3.5
- net PWM16: now also R9.4; no longer R3.5
- net PWM17: now also R9.3; no longer R3.6
- net PWM18: now also R9.2; no longer R3.7
- net PWM19: now also R9.1; no longer R3.8
- net PWM2: now also R6.6; no longer R6.7
- net PWM20: now also R10.4; no longer R2.5
- net PWM21: now also R10.3; no longer R2.6
- net PWM22: no longer R2.7
- net PWM23: now also R10.1; no longer R2.8
- net PWM24: no longer R1.5
- net PWM25: no longer R1.6
- net PWM26: no longer R1.7
- net PWM27: no longer R1.8
- net PWM3: now also R6.5; no longer R6.8
- net PWM4: now also R5.8; no longer R5.5
- net PWM5: now also R5.7; no longer R5.6
- net PWM6: now also R5.6; no longer R5.7
- net PWM7: now also R5.5; no longer R5.8
- net PWM8: now also R4.8; no longer R4.5
- net PWM9: now also R4.7; no longer R4.6
Routing:
- net SCL: track 0.00 -> 36.4 mm
- net SDA: track 0.00 -> 24.7 mm
- net +5V: track 0.00 -> 17.1 mm
- net N$7: track 0.00 -> 6.70 mm
- net N$6: track 0.00 -> 6.70 mm
- net N$30: track 0.00 -> 6.70 mm
- net N$27: track 0.00 -> 6.70 mm

Commit message: Working on PCB
Parts:
- added C1: 100nF, capacitor-wima:C2.5-3
- added C2, C3: 22p, capacitor-wima:C2.5-3
- added Q1: 12MHz, crystal:CSM-7X-DU
- added U4: CH340G, HumanoidLbr:SO-16
- added X1: MINI-USB-UX60-MB-5S8, con-hirose:UX60-MB-5S8
- moved JP9 65.6 mm to (88.9, 3.81), turned to 270 degrees
- moved S1 56.1 mm to (96.5, 7.62), turned to 180 degrees
- moved J2 55.2 mm to (78.7, 5.08)
- moved U1 54.9 mm to (22.9, 10.2), turned to 180 degrees
- moved U$3 50.3 mm to (31.8, 63.5), turned to 180 degrees
- moved U$1 48.6 mm to (90.2, 10.2), turned to 90 degrees
- moved R3 30.0 mm to (21.6, 27.9)
- moved R4 28.5 mm to (21.6, 34.3)
- moved R5 27.3 mm to (21.6, 40.6)
- moved R9 27.1 mm to (80.0, 27.9)
- moved R6 26.7 mm to (21.6, 45.7)
- moved U$2 26.2 mm to (90.2, 15.2), turned to 0 degrees
- moved R10 25.9 mm to (80.0, 33.0)
- moved R8 25.7 mm to (88.9, 19.1), turned to 180 degrees
- moved R7 24.5 mm to (74.9, 19.1)
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Connections:
- new net D+: U4.5, X1.3
- new net D-: U4.6, X1.2
- new net N$56: C2.1, Q1.2, U4.7
- new net N$57: C3.1, Q1.1, U4.8
- new net RX: U$3.UART1-TX, U4.3
- new net TX: U$3.UART1-RX, U4.2
- net +5V: now also C1.1, U4.16, X1.1
- net GND: now also C1.2, C2.2, C3.2, U4.1, X1.5
Routing:
- net SCL: track 36.4 -> 0.00 mm
- net SDA: track 24.7 -> 0.00 mm
Other:
- board size 105.4 x 75.2 mm -> 100 x 65 mm

Commit message: Added boost circuit for charging
Parts:
- added C4: 22p, capacitor-wima:C2.5-3
- added D1: HSMS-285B, avago:SOT323
- added L1: (no value), inductor-neosid:SM-1206
- added R11, R12: 670R, SparkFun-Passives:0805
- added U5: SX1308_B628, HumanoidLbr:SOT23-6
- moved U2 3.81 mm to (80.0, 59.7)
Connections:
- new net N$58: L1.1, U5.P$4, U5.P$5
- new net N$59: R12.2, U5.P$3
- new net N$60: C4.1, D1.1, L1.2, R11.2, U5.P$1
- new net V-CHG: D1.3
- net GND: now also C4.2, R12.1, U5.P$2
