File: PCBA/Head/Head.brd (EAGLE design)
At the start: 2 x 8.3 mm, 10 parts, among them IC2 ATMEGA325P, U1 CH340G, X1 MINI-USB_SHIELD5P2-32005-601

Commit message: Added frame to head PCBA
Make it look gewd.
Parts:
- moved U1 149.2 mm to (92.7, 30.5)
- moved X1 130.6 mm to (26.7, 53.3)
- moved IC2 123.6 mm to (15.2, 19.1)
- moved D5 106.4 mm to (54.6, 33.0)
- moved D1 106.4 mm to (54.6, 68.6)
- moved D2 106.4 mm to (54.6, 59.7)
- moved D3 106.4 mm to (54.6, 50.8)
- moved D4 106.4 mm to (54.6, 41.9)
- moved D6 106.4 mm to (54.6, 24.1)
- moved D7 106.4 mm to (54.6, 15.2)
Connections:
- removed net VDD: D1.1, D2.1, D3.1, D4.1, D5.1, D6.1, D7.1
- new net 0V: D1.3, D2.3, D3.3, D4.3, D5.3, D6.3, D7.3
- new net N$1: D1.2, D2.4
- new net N$2: D2.2, D3.4
- new net N$3: D3.2, D4.4
- new net N$4: D4.2, D5.4
- new net N$5: D5.2, D6.4
- new net N$6: D6.2, D7.4
- new net N$7: D1.4, IC2.49
- net VCC: now also D1.1, D2.1, D3.1, D4.1, D5.1, D6.1, D7.1
