File: PCBA/Head/Head.sch (EAGLE design)
At the start: 10 parts, among them IC2 ATMEGA325P, U1 CH340G, X1 MINI-USB_SHIELD5P2-32005-601

Commit message: Added frame to head PCBA
Make it look gewd.
Connections:
- new net 0V: D1.VSS, D2.VSS, D3.VSS, D4.VSS, D5.VSS, D6.VSS, D7.VSS
- new net N$1: D1.DOUT, D2.DIN
- new net N$2: D2.DOUT, D3.DIN
- new net N$3: D3.DOUT, D4.DIN
- new net N$4: D4.DOUT, D5.DIN
- new net N$5: D5.DOUT, D6.DIN
- new net N$6: D6.DOUT, D7.DIN
- new net N$7: D1.DIN, IC2.PA2
- new net VCC: D1.VDD, D2.VDD, D3.VDD, D4.VDD, D5.VDD, D6.VDD, D7.VDD
Other:
- moved on the sheet: D1, D2, D3, D4, D5, D6, D7, IC2, U1, X1
Changed lines of the file:
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@@
 <part name="X1" library="con-cypressindustries" deviceset="MINI-USB_SHIELD5P2-" device="32005-601"/>
 <part name="IC2" library="atmel" deviceset="ATMEGA325P" device=""/>
+<part name="FRAME1" library="frames" deviceset="A3L-LOC" device=""/>
+<part name="P+1" library="supply1" deviceset="VCC" device="" value="+5V"/>
+<part name="P+2" library="supply1" deviceset="VCC" device="" value="+5V"/>
+<part name="P+3" library="supply1" deviceset="VCC" device="" value="+5V"/>
+<part name="P+4" library="supply1" deviceset="VCC" device="" value="+5V"/>
+<part name="P+5" library="supply1" deviceset="VCC" device="" value="+5V"/>
+<part name="P+6" library="supply1" deviceset="VCC" device="" value="+5V"/>
+<part name="P+7" library="supply1" deviceset="VCC" device="" value="+5V"/>
+<part name="GND1" library="supply1" deviceset="0V" device="" value="GND"/>
+<part name="GND2" library="supply1" deviceset="0V" device="" value="GND"/>
+<part name="GND3" library="supply1" deviceset="0V" device="" value="GND"/>
+<part name="GND4" library="supply1" deviceset="0V" device="" value="GND"/>
+<part name="GND5" library="supply1" deviceset="0V" device="" value="GND"/>
+<part name="GND6" library="supply1" deviceset="0V" device="" value="GND"/>
+<part name="GND7" library="supply1" deviceset="0V" device="" value="GND"/>
 </parts>
 <sheets>
@@
 </plain>
 <instances>
-<instance part="D1" gate="G$1" x="30.48" y="27.94"/>
-<instance part="D2" gate="G$1" x="68.58" y="27.94"/>
-<instance part="D3" gate="G$1" x="106.68" y="27.94"/>
-<instance part="D4" gate="G$1" x="144.78" y="27.94"/>
-<instance part="D5" gate="G$1" x="187.96" y="27.94"/>
-<instance part="D6" gate="G$1" x="228.6" y="27.94"/>
-<instance part="D7" gate="G$1" x="269.24" y="27.94"/>
-<instance part="U1" gate="G$1" x="40.64" y="73.66"/>
-<instance part="X1" gate="G41" x="38.1" y="160.02"/>
-<instance part="IC2" gate="G$1" x="154.94" y="101.6"/>
+<instance part="D1" gate="G$1" x="119.38" y="93.98"/>
+<instance part="D2" gate="G$1" x="157.48" y="93.98"/>
+<instance part="D3" gate="G$1" x="195.58" y="93.98"/>
+<instance part="D4" gate="G$1" x="233.68" y="93.98"/>
+<instance part="D5" gate="G$1" x="276.86" y="93.98"/>
+<instance part="D6" gate="G$1" x="317.5" y="93.98"/>
+<instance part="D7" gate="G$1" x="358.14" y="93.98"/>
+<instance part="U1" gate="G$1" x="40.64" y="35.56"/>
+<instance part="X1" gate="G41" x="17.78" y="109.22" rot="R180"/>
+<instance part="IC2" gate="G$1" x="109.22" y="38.1"/>
+<instance part="FRAME1" gate="G$1" x="0" y="0"/>
+<instance part="P+1" gate="VCC" x="137.16" y="106.68"/>
+<instance part="P+2" gate="VCC" x="175.26" y="106.68"/>
+<instance part="P+3" gate="VCC" x="213.36" y="106.68"/>
+<instance part="P+4" gate="VCC" x="251.46" y="106.68"/>
+<instance part="P+5" gate="VCC" x="294.64" y="106.68"/>
+<instance part="P+6" gate="VCC" x="335.28" y="106.68"/>
+<instance part="P+7" gate="VCC" x="375.92" y="106.68"/>
+<instance part="GND1" gate="1" x="134.62" y="83.82"/>
+<instance part="GND2" gate="1" x="172.72" y="83.82"/>
+<instance part="GND3" gate="1" x="210.82" y="83.82"/>
+<instance part="GND4" gate="1" x="248.92" y="83.82"/>
+<instance part="GND5" gate="1" x="292.1" y="83.82"/>
+<instance part="GND6" gate="1" x="332.74" y="83.82"/>
+<instance part="GND7" gate="1" x="373.38" y="83.82"/>
 </instances>
 <busses>
 </busses>
 <nets>
+<net name="N$1" class="0">
+<segment>
+<pinref part="D1" gate="G$1" pin="DOUT"/>
+<pinref part="D2" gate="G$1" pin="DIN"/>
+<wire x1="134.62" y1="93.98" x2="142.24" y2="93.98" width="0.1524" layer="91"/>
+</segment>
+</net>
+<net name="N$2" class="0">
+<segment>
+<pinref part="D2" gate="G$1" pin="DOUT"/>
+<pinref part="D3" gate="G$1" pin="DIN"/>
+<wire x1="172.72" y1="93.98" x2="180.34" y2="93.98" width="0.1524" layer="91"/>
+</segment>
+</net>
+<net name="N$3" class="0">
+<segment>
+<pinref part="D3" gate="G$1" pin="DOUT"/>
+<pinref part="D4" gate="G$1" pin="DIN"/>
+<wire x1="210.82" y1="93.98" x2="218.44" y2="93.98" width="0.1524" layer="91"/>
+</segment>
+</net>
+<net name="N$4" class="0">
+<segment>
+<pinref part="D4" gate="G$1" pin="DOUT"/>
+<pinref part="D5" gate="G$1" pin="DIN"/>
+<wire x1="248.92" y1="93.98" x2="261.62" y2="93.98" width="0.1524" layer="91"/>
+</segment>
+</net>
+<net name="N$5" class="0">
+<segment>
+<pinref part="D5" gate="G$1" pin="DOUT"/>
+<pinref part="D6" gate="G$1" pin="DIN"/>
+<wire x1="292.1" y1="93.98" x2="302.26" y2="93.98" width="0.1524" layer="91"/>
+</segment>
+</net>
+<net name="N$6" class="0">
+<segment>
+<pinref part="D6" gate="G$1" pin="DOUT"/>
+<pinref part="D7" gate="G$1" pin="DIN"/>
+<wire x1="332.74" y1="93.98" x2="342.9" y2="93.98" width="0.1524" layer="91"/>
+</segment>
+</net>
+<net name="VCC" class="0">
+<segment>
+<pinref part="P+7" gate="VCC" pin="VCC"/>
+<pinref part="D7" gate="G$1" pin="VDD"/>
+<wire x1="375.92" y1="104.14" x2="375.92" y2="101.6" width="0.1524" layer="91"/>
+<wire x1="375.92" y1="101.6" x2="373.38" y2="101.6" width="0.1524" layer="91"/>
+</segment>
+<segment>
+<pinref part="D6" gate="G$1" pin="VDD"/>
+<pinref part="P+6" gate="VCC" pin="VCC"/>
+<wire x1="332.74" y1="101.6" x2="335.28" y2="101.6" width="0.1524" layer="91"/>
+<wire x1="335.28" y1="101.6" x2="335.28" y2="104.14" width="0.1524" layer="91"/>
+</segment>
+<segment>
+<pinref part="D5" gate="G$1" pin="VDD"/>
+<pinref part="P+5" gate="VCC" pin="VCC"/>
+<wire x1="292.1" y1="101.6" x2="294.64" y2="101.6" width="0.1524" layer="91"/>
+<wire x1="294.64" y1="101.6" x2="294.64" y2="104.14" width="0.1524" layer="91"/>
+</segment>
+<segment>
+<pinref part="D4" gate="G$1" pin="VDD"/>
+<pinref part="P+4" gate="VCC" pin="VCC"/>
+<wire x1="248.92" y1="101.6" x2="251.46" y2="101.6" width="0.1524" layer="91"/>
+<wire x1="251.46" y1="101.6" x2="251.46" y2="104.14" width="0.1524" layer="91"/>
+</segment>
+<segment>
+<pinref part="D3" gate="G$1" pin="VDD"/>
+<pinref part="P+3" gate="VCC" pin="VCC"/>
+<wire x1="210.82" y1="101.6" x2="213.36" y2="101.6" width="0.1524" layer="91"/>
+<wire x1="213.36" y1="101.6" x2="213.36" y2="104.14" width="0.1524" layer="91"/>
+</segment>
+<segment>
+<pinref part="D2" gate="G$1" pin="VDD"/>
+<pinref part="P+2" gate="VCC" pin="VCC"/>
+<wire x1="172.72" y1="101.6" x2="175.26" y2="101.6" width="0.1524" layer="91"/>
+<wire x1="175.26" y1="101.6" x2="175.26" y2="104.14" width="0.1524" layer="91"/>
+</segment>
+<segment>
+<pinref part="D1" gate="G$1" pin="VDD"/>
+<pinref part="P+1" gate="VCC" pin="VCC"/>
+<wire x1="134.62" y1="101.6" x2="137.16" y2="101.6" width="0.1524" layer="91"/>
+<wire x1="137.16" y1="101.6" x2="137.16" y2="104.14" width="0.1524" layer="91"/>
+</segment>
+</net>
+<net name="0V" class="0">
+<segment>
+<pinref part="D1" gate="G$1" pin="VSS"/>
+<pinref part="GND1" gate="1" pin="0V"/>
+</segment>
+<segment>
+<pinref part="D2" gate="G$1" pin="VSS"/>
+<pinref part="GND2" gate="1" pin="0V"/>
+</segment>
+<segment>
+<pinref part="D3" gate="G$1" pin="VSS"/>
+<pinref part="GND3" gate="1" pin="0V"/>
+</segment>
+<segment>
+<pinref part="D4" gate="G$1" pin="VSS"/>
+<pinref part="GND4" gate="1" pin="0V"/>
+</segment>
+<segment>
+<pinref part="D5" gate="G$1" pin="VSS"/>
+<pinref part="GND5" gate="1" pin="0V"/>
+</segment>
+<segment>
+<pinref part="D6" gate="G$1" pin="VSS"/>
+<pinref part="GND6" gate="1" pin="0V"/>
+</segment>
+<segment>
+<pinref part="D7" gate="G$1" pin="VSS"/>
+<pinref part="GND7" gate="1" pin="0V"/>
+</segment>
+</net>
+<net name="N$7" class="0">
+<segment>
+<pinref part="IC2" gate="G$1" pin="PA2"/>
+<wire x1="132.08" y1="66.04" x2="132.08" y2="76.2" width="0.1524" layer="91"/>
+<wire x1="132.08" y1="76.2" x2="104.14" y2="76.2" width="0.1524" layer="91"/>
+<pinref part="D1" gate="G$1" pin="DIN"/>
+<wire x1="104.14" y1="76.2" x2="104.14" y2="93.98" width="0.1524" layer="91"/>
+</segment>
+</net>
 </nets>
 </sheet>
